File: HW/Badge-OWASP-2020/Badge-OWASP-2020.sch (KiCad schematic (older format))
At the start: 28 parts, among them J1 Shitty Add-Ons, J2 Battery, J3 I2C, J4 USB_B, Q1 MMBT3904, Q2 DMG3415U-7, Q3 MMBT3904, SW1 RST, SW2 BOOT, U1 ESP32-WROOM-32, U2 CH340C, U3 AP111733

Commit message: Add manf#
Parts:
- C1, C2, C3: lscs# (none) -> C376923; manf# (none) -> TCC0805X7R104K250DTS
- C4, C5: lscs# (none) -> C385902; manf# (none) -> EMK212BJ475KG-T
- D1, D2: lscs# (none) -> C114583; manf# (none) -> WS2812B-Mini
- D3: lscs# (none) -> C130880; manf# (none) -> MBR120LSF
- F1: lscs# (none) -> C369166; manf# (none) -> JK-MSMD030
- J1, J2, J3: lscs# (none) -> -; manf# (none) -> -
- J4: lscs# (none) -> C319170; manf# (none) -> U254-051N-4BH806
- Q1, Q3: lscs# (none) -> C181119; manf# (none) -> MMBT3904
- Q2: symbol Transistor_FET:DMG2301L -> Badge-OWASP-2020-rescue:DMG2301L-Transistor_FET; lscs# (none) -> C96616; manf# (none) -> DMG3415U-7
- R1, R3, R4, R5, R6: lscs# (none) -> C25612; manf# (none) -> 0805W8J0103T5E
- R2: lscs# (none) -> C119076; manf# (none) -> RS-05K471JT
- R7: lscs# (none) -> C118844; manf# (none) -> RS-05K104JT
- SW1, SW2: lscs# (none) -> C318893; manf# (none) -> TS-1185EC-C-D-B
- U1: lscs# (none) -> -; manf# (none) -> ESP32-WROOM-32
- U2: lscs# (none) -> C84681; manf# (none) -> CH340C
- U3: value AP111733 -> AP1117; lscs# (none) -> C108785; manf# (none) -> AP1117E33G-13
Changed lines of the file:
@@
 EESchema Schematic File Version 4
 LIBS:Badge-OWASP-2020-cache
-EELAYER 30 0
+EELAYER 29 0
 EELAYER END
 $Descr A4 11693 8268
@@
 F 2 "Package_SO:SOIC-16_3.9x9.9mm_P1.27mm" H 9900 5000 50  0001 L CNN
 F 3 "http://www.datasheet5.com/pdf-local-2195953" H 9500 6350 50  0001 C CNN
+F 4 "CH340C" H 0   0   50  0001 C CNN "manf#"
+F 5 "C84681" H 0   0   50  0001 C CNN "lscs#"
 	1    9850 5550
 	1    0    0    -1
@@
 P 2400 6920
 F 0 "U3" H 2400 7162 50  0000 C CNN
-F 1 "AP111733" H 2400 7071 50  0000 C CNN
+F 1 "AP1117" H 2400 7071 50  0000 C CNN
 F 2 "Package_TO_SOT_SMD:SOT-223-3_TabPin2" H 2400 7120 50  0001 C CNN
 F 3 "http://www.diodes.com/datasheets/AP1117.pdf" H 2500 6670 50  0001 C CNN
+F 4 "AP1117E33G-13" H 0   0   50  0001 C CNN "manf#"
+F 5 "C108785" H 0   0   50  0001 C CNN "lscs#"
 	1    2400 6920
 	1    0    0    -1
@@
 F 2 "Capacitor_SMD:C_0805_2012Metric_Pad1.15x1.40mm_HandSolder" H 2888 7070 50  0001 C CNN
 F 3 "~" H 2850 7220 50  0001 C CNN
+F 4 "C385902" H 0   0   50  0001 C CNN "lscs#"
+F 5 "EMK212BJ475KG-T" H 0   0   50  0001 C CNN "manf#"
 	1    2850 7220
 	1    0    0    -1
@@
 F 2 "Capacitor_SMD:C_0805_2012Metric_Pad1.15x1.40mm_HandSolder" H 2038 7120 50  0001 C CNN
 F 3 "~" H 2000 7270 50  0001 C CNN
+F 4 "C385902" H 0   0   50  0001 C CNN "lscs#"
+F 5 "EMK212BJ475KG-T" H 0   0   50  0001 C CNN "manf#"
 	1    2000 7270
 	1    0    0    -1
@@
 F 2 "Diode_SMD:D_SOD-123F" H 1540 6920 50  0001 C CNN
 F 3 "~" H 1540 6920 50  0001 C CNN
+F 4 "MBR120LSF" H 0   0   50  0001 C CNN "manf#"
+F 5 "C130880" H 1540 6920 50  0001 C CNN "lscs#"
 	1    1540 6920
 	-1   0    0    1
@@
 F 2 "Package_TO_SOT_SMD:SOT-23" H 5800 6375 50  0001 L CIN
 F 3 "https://www.fairchildsemi.com/datasheets/2N/2N3904.pdf" H 5600 6450 50  0001 L CNN
+F 4 "MMBT3904" H 0   0   50  0001 C CNN "manf#"
+F 5 "C181119" H 0   0   50  0001 C CNN "lscs#"
 	1    5600 6450
 	1    0    0    -1
@@
 F 2 "Package_TO_SOT_SMD:SOT-23" H 5800 6975 50  0001 L CIN
 F 3 "https://www.fairchildsemi.com/datasheets/2N/2N3904.pdf" H 5600 7050 50  0001 L CNN
+F 4 "MMBT3904" H 0   0   50  0001 C CNN "manf#"
+F 5 "C181119" H 0   0   50  0001 C CNN "lscs#"
 	1    5600 7050
 	1    0    0    -1
@@
 F 2 "Resistor_SMD:R_0805_2012Metric_Pad1.15x1.40mm_HandSolder" V 4930 6450 50  0001 C CNN
 F 3 "~" H 5000 6450 50  0001 C CNN
+F 4 "0805W8J0103T5E" H 0   0   50  0001 C CNN "manf#"
+F 5 "C25612" H 0   0   50  0001 C CNN "lscs#"
 	1    5000 6450
 	0    1    1    0
@@
 F 2 "Resistor_SMD:R_0805_2012Metric_Pad1.15x1.40mm_HandSolder" V 4930 7050 50  0001 C CNN
 F 3 "~" H 5000 7050 50  0001 C CNN
+F 4 "0805W8J0103T5E" H 0   0   50  0001 C CNN "manf#"
+F 5 "C25612" H 0   0   50  0001 C CNN "lscs#"
 	1    5000 7050
 	0    1    1    0
@@
 F 2 "LED_SMD:LED_SK6812MINI_PLCC4_3.5x3.5mm_P1.75mm" H 1450 1700 50  0001 L TNN
 F 3 "https://cdn-shop.adafruit.com/datasheets/WS2812B.pdf" H 1500 1625 50  0001 L TNN
+F 4 "WS2812B-Mini" H 0   0   50  0001 C CNN "manf#"
+F 5 "C114583" H 0   0   50  0001 C CNN "lscs#"
 	1    1400 2000
 	1    0    0    -1
@@
 F 2 "LED_SMD:LED_SK6812MINI_PLCC4_3.5x3.5mm_P1.75mm" H 2500 1700 50  0001 L TNN
 F 3 "https://cdn-shop.adafruit.com/datasheets/WS2812B.pdf" H 2550 1625 50  0001 L TNN
+F 4 "WS2812B-Mini" H 0   0   50  0001 C CNN "manf#"
+F 5 "C114583" H 0   0   50  0001 C CNN "lscs#"
 	1    2450 2000
 	1    0    0    -1
@@
 F 2 "Capacitor_SMD:C_0805_2012Metric_Pad1.15x1.40mm_HandSolder" H 2838 2700 50  0001 C CNN
 F 3 "~" H 2800 2850 50  0001 C CNN
+F 4 "C376923" H 0   0   50  0001 C CNN "lscs#"
+F 5 "TCC0805X7R104K250DTS" H 0   0   50  0001 C CNN "manf#"
 	1    2800 2850
 	1    0    0    -1
@@
 F 2 "Connector_PinHeader_2.54mm:PinHeader_1x04_P2.54mm_Vertical" H 2050 5150 50  0001 C CNN
 F 3 "~" H 2050 5150 50  0001 C CNN
+F 4 "-" H 0   0   50  0001 C CNN "manf#"
+F 5 "-" H 0   0   50  0001 C CNN "lscs#"
 	1    2050 5150
 	1    0    0    -1
@@
 F 2 "Resistor_SMD:R_0805_2012Metric_Pad1.15x1.40mm_HandSolder" V 1030 5050 50  0001 C CNN
 F 3 "~" H 1100 5050 50  0001 C CNN
+F 4 "0805W8J0103T5E" V 1100 5050 50  0001 C CNN "manf#"
+F 5 "C25612" H 0   0   50  0001 C CNN "lscs#"
 	1    1100 5050
 	-1   0    0    1
@@
 F 2 "Resistor_SMD:R_0805_2012Metric_Pad1.15x1.40mm_HandSolder" V 1430 5000 50  0001 C CNN
 F 3 "~" H 1500 5000 50  0001 C CNN
+F 4 "0805W8J0103T5E" H 0   0   50  0001 C CNN "manf#"
+F 5 "C25612" H 0   0   50  0001 C CNN "lscs#"
 	1    1500 5000
 	-1   0    0    1
@@
 F 2 "RF_Module:ESP32-WROOM-32" H 6155 1080 50  0001 C CNN
 F 3 "https://www.espressif.com/sites/default/files/documentation/esp32-wroom-32_datasheet_en.pdf" H 5855 2630 50  0001 C CNN
+F 4 "ESP32-WROOM-32" H 0   0   50  0001 C CNN "manf#"
+F 5 "-" H 0   0   50  0001 C CNN "lscs#"
 	1    6155 2580
 	1    0    0    -1
@@
 F 2 "Fuse:Fuse_1812_4532Metric_Pad1.30x3.40mm_HandSolder" V 7880 5200 50  0001 C CNN
 F 3 "~" H 7950 5200 50  0001 C CNN
+F 4 "JK-MSMD030" H 0   0   50  0001 C CNN "manf#"
+F 5 "C369166" H 0   0   50  0001 C CNN "lscs#"
 	1    7950 5200
 	0    1    1    0
@@
 F 2 "Connector_USB:USB_Micro-B_Wuerth_629105150521" H 7550 5350 50  0001 C CNN
 F 3 " ~" H 7550 5350 50  0001 C CNN
+F 4 "C319170" H 0   0   50  0001 C CNN "lscs#"
+F 5 "U254-051N-4BH806" H 0   0   50  0001 C CNN "manf#"
 	1    7400 5400
 	1    0    0    -1
@@
 F 2 "Capacitor_SMD:C_0805_2012Metric_Pad1.15x1.40mm_HandSolder" H 1688 2700 50  0001 C CNN
 F 3 "~" H 1650 2850 50  0001 C CNN
+F 4 "C376923" H 0   0   50  0001 C CNN "lscs#"
+F 5 "TCC0805X7R104K250DTS" H 0   0   50  0001 C CNN "manf#"
 	1    1650 2850
 	1    0    0    -1
@@
 F 2 "Capacitor_SMD:C_0805_2012Metric_Pad1.15x1.40mm_HandSolder" H 8108 2370 50  0001 C CNN
 F 3 "~" H 8070 2520 50  0001 C CNN
+F 4 "C376923" H 0   0   50  0001 C CNN "lscs#"
+F 5 "TCC0805X7R104K250DTS" H 0   0   50  0001 C CNN "manf#"
 	1    8070 2520
 	1    0    0    -1
@@
 F 2 "Resistor_SMD:R_0805_2012Metric_Pad1.15x1.40mm_HandSolder" V 7135 2280 50  0001 C CNN
 F 3 "~" H 7205 2280 50  0001 C CNN
+F 4 "C119076" H 0   0   50  0001 C CNN "lscs#"
+F 5 "RS-05K471JT" H 0   0   50  0001 C CNN "manf#"
 	1    7205 2280
 	0    1    1    0
@@
 F 2 "Button_Switch_SMD:SW_SPST_TL3342" H 4605 2180 50  0001 C CNN
 F 3 "~" H 4605 2180 50  0001 C CNN
+F 4 "C318893" H 0   0   50  0001 C CNN "lscs#"
+F 5 "TS-1185EC-C-D-B" H 0   0   50  0001 C CNN "manf#"
 	1    4605 1980
 	1    0    0    -1
@@
 F 2 "Button_Switch_SMD:SW_SPST_TL3342" H 4605 3530 50  0001 C CNN
 F 3 "~" H 4605 3530 50  0001 C CNN
+F 4 "C318893" H 0   0   50  0001 C CNN "lscs#"
+F 5 "TS-1185EC-C-D-B" H 0   0   50  0001 C CNN "manf#"
 	1    4605 3330
 	1    0    0    -1
@@
 F 2 "Resistor_SMD:R_0805_2012Metric_Pad1.15x1.40mm_HandSolder" V 5085 1230 50  0001 C CNN
 F 3 "~" H 5155 1230 50  0001 C CNN
+F 4 "0805W8J0103T5E" H 0   0   50  0001 C CNN "manf#"
+F 5 "C25612" H 0   0   50  0001 C CNN "lscs#"
 	1    5155 1230
 	-1   0    0    1
@@
 F 2 "Connector_PinHeader_2.54mm:PinHeader_1x02_P2.54mm_Vertical" H 5505 5105 50  0001 C CNN
 F 3 "~" H 5505 5105 50  0001 C CNN
+F 4 "-" H 0   0   50  0001 C CNN "manf#"
+F 5 "-" H 0   0   50  0001 C CNN "lscs#"
 	1    5505 5105
 	1    0    0    -1
@@
 $EndComp
 $Comp
-L Transistor_FET:DMG2301L Q2
+L Badge-OWASP-2020-rescue:DMG2301L-Transistor_FET Q2
 U 1 1 5E039884
 P 1705 6660
 F 0 "Q2" H 1911 6706 50  0000 L CNN
-F 1 "DMG3415U-7" H 1860 6775 50  0000 L CNN
+F 1 "DMG3415U-7" H 1925 6800 50  0000 L CNN
 F 2 "Package_TO_SOT_SMD:SOT-23" H 1905 6585 50  0001 L CIN
 F 3 "https://www.diodes.com/assets/Datasheets/DMG2301L.pdf" H 1705 6660 50  0001 L CNN
+F 4 "DMG3415U-7" H 0   0   50  0001 C CNN "manf#"
+F 5 "C96616" H 0   0   50  0001 C CNN "lscs#"
 	1    1705 6660
 	1    0    0    -1
@@
 F 2 "Resistor_SMD:R_0805_2012Metric_Pad1.15x1.40mm_HandSolder" H 1350 7095 50  0001 C CNN
 F 3 "~" H 1350 7095 50  0001 C CNN
+F 4 "C118844" H 0   0   50  0001 C CNN "lscs#"
+F 5 "RS-05K104JT" H 0   0   50  0001 C CNN "manf#"
 	1    1350 7095
 	1    0    0    -1
@@
 F 2 "Connector_PinHeader_2.54mm:PinHeader_2x03_P2.54mm_Vertical" H 10040 2330 50  0001 C CNN
 F 3 "~" H 10040 2330 50  0001 C CNN
+F 4 "-" H 0   0   50  0001 C CNN "manf#"
+F 5 "-" H 0   0   50  0001 C CNN "lscs#"
 	1    10040 2330
 	0    -1   1    0

Commit message: fix names tx and rx drc
Connections:
- net RXD is gone; now on net RX: U2.3 (RXD)
- net TXD is gone; now on net TX: U2.2 (TXD)
- no-connect marks 29 -> 31
Changed lines of the file:
@@
 EESchema Schematic File Version 4
 LIBS:Badge-OWASP-2020-cache
-EELAYER 29 0
+EELAYER 30 0
 EELAYER END
 $Descr A4 11693 8268
@@
 Comment4 ""
 $EndDescr
-$Comp
-L Badge-OWASP-2020-rescue:CH340C-Interface_USB2 U2
-U 1 1 5DF1A7B6
-P 9850 5550
-F 0 "U2" H 9450 5050 50  0000 C CNN
-F 1 "CH340C" H 9550 4900 50  0000 C CNN
-F 2 "Package_SO:SOIC-16_3.9x9.9mm_P1.27mm" H 9900 5000 50  0001 L CNN
-F 3 "http://www.datasheet5.com/pdf-local-2195953" H 9500 6350 50  0001 C CNN
-F 4 "CH340C" H 0   0   50  0001 C CNN "manf#"
-F 5 "C84681" H 0   0   50  0001 C CNN "lscs#"
-	1    9850 5550
-	1    0    0    -1
-$EndComp
 Text Label 10250 5150 0    50   ~ 0
-TXD
+TX
 Text Label 10250 5250 0    50   ~ 0
-RXD
+RX
 Text Label 10250 5950 0    50   ~ 0
 RTS
@@
 Text Notes 9965 850  0    50   ~ 0
 sao1.69bis
+NoConn ~ 5555 2580
+$Comp
+L Badge-OWASP-2020-rescue:CH340C-Interface_USB2 U2
+U 1 1 5DF1A7B6
+P 9850 5550
+F 0 "U2" H 9450 5050 50  0000 C CNN
+F 1 "CH340C" H 9550 4900 50  0000 C CNN
+F 2 "Package_SO:SOIC-16_3.9x9.9mm_P1.27mm" H 9900 5000 50  0001 L CNN
+F 3 "http://www.datasheet5.com/pdf-local-2195953" H 9500 6350 50  0001 C CNN
+F 4 "CH340C" H 0   0   50  0001 C CNN "manf#"
+F 5 "C84681" H 0   0   50  0001 C CNN "lscs#"
+	1    9850 5550
+	1    0    0    -1
+$EndComp
+NoConn ~ 10250 5650
 $EndSCHEMATC

Commit message: Add USB connector from LCSC change angle of components
Parts:
- removed J4: USB_B, Connector_USB:USB_Micro-B_Wuerth_629105150521, symbol Connector:USB_B
- added J4: USB_B_Micro, Connectors:U254051N4BH806, symbol Connector:USB_B_Micro
Connections:
- net D+: now also J4.3 (D+)
- net D-: now also J4.2 (D-)
- net GND: now also J4.5 (GND), J4.6 (Shield)
- net at F1.2: now also J4.1 (VBUS)
- no-connect marks 31 -> 32
Changed lines of the file:
@@
 EESchema Schematic File Version 4
 LIBS:Badge-OWASP-2020-cache
-EELAYER 30 0
+EELAYER 29 0
 EELAYER END
 $Descr A4 11693 8268
@@
 Sheet 1 1
 Title "OWASP badge"
-Date "2019-12-11"
+Date "2020-01-09"
 Rev "1.0"
 Comp "Electronic Cats"
@@
 Wire Wire Line
 	7300 6100 7300 5950
-$Comp
-L Connector:USB_B J4
-U 1 1 5DF2C252
-P 7400 5400
-F 0 "J4" H 7457 5867 50  0000 C CNN
-F 1 "USB_B" H 7457 5776 50  0000 C CNN
-F 2 "Connector_USB:USB_Micro-B_Wuerth_629105150521" H 7550 5350 50  0001 C CNN
-F 3 " ~" H 7550 5350 50  0001 C CNN
-F 4 "C319170" H 0   0   50  0001 C CNN "lscs#"
-F 5 "U254-051N-4BH806" H 0   0   50  0001 C CNN "manf#"
-	1    7400 5400
-	1    0    0    -1
-$EndComp
 Wire Notes Line
 	6950 6550 6950 4450
@@
 $EndComp
 NoConn ~ 10250 5650
+$Comp
+L Connector:USB_B_Micro J4
+U 1 1 5E1CB56D
+P 7400 5400
+F 0 "J4" H 7457 5867 50  0000 C CNN
+F 1 "USB_B_Micro" H 7457 5776 50  0000 C CNN
+F 2 "Connectors:U254051N4BH806" H 7550 5350 50  0001 C CNN
+F 3 "~" H 7550 5350 50  0001 C CNN
+	1    7400 5400
+	1    0    0    -1
+$EndComp
+NoConn ~ 7700 5600
 $EndSCHEMATC
