File: HW/Badge-OWASP-2020/Badge-OWASP-2020.kicad_pcb (KiCad board)
At the start: 2 copper layers, 98.6 x 65.9 mm, 33 parts, among them J1 Shitty Add-Ons, J2 Battery, J3 I2C, J4 USB_B_Micro, Q1 MMBT3904, Q2 DMG3415U-7, Q3 MMBT3904, SW1 RST, SW2 BOOT, U1 ESP32-WROOM-32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

Commit message: Update buttons
Parts:
- moved SW2 59.6 mm to (167.7, 89.0)
- moved SW1 44.8 mm to (182.3, 84.5), turned to 226 degrees
- moved J3 12.2 mm to (119.6, 49.7), turned to 156 degrees
- turned R3 to 180 degrees
- turned R4 to 180 degrees
Routing:
- net /EN: track 30.5 -> 86.7 mm
- net /GPIO0: track 47.6 -> 87.7 mm
- net GND: track 180.6 -> 149.4 mm, vias 19 -> 18
- net +3V3: track 183.6 -> 197.9 mm, vias 6 -> 4
- net /SDA: track 48.2 -> 35.0 mm, vias 1 -> 0
- net /GPIO2: track 20.3 -> 33.4 mm, vias 0 -> 2
- net /TX: track 43.6 -> 56.2 mm
- net /RX: track 44.4 -> 56.6 mm
- net /GPIO1: track 48.4 -> 59.8 mm, vias 1 -> 2
- net /RTS: track 22.3 -> 24.7 mm
- net /NP: track 9.78 -> 8.61 mm
- net /SCL: track 38.0 -> 38.3 mm, vias 1 -> 2
